Commit message: added mujuco and isaac

File: src/base101_control/urdf/base101.hardware.xacro (robot description, xacro)
@@ -2,9 +2,9 @@
 <robot name="base101" xmlns:xacro="http://www.ros.org/wiki/xacro">
   <xacro:arg name="variant" default="simple"/>
-  <!-- Force-disable the sim ros2_control + gazebo extensions so this URDF is
+  <!-- Force-disable the sim ros2_control + per-sim extensions so this URDF is
        safe to load on real hardware. Xacro takes the first <xacro:arg> for a
-       given name, so declaring use_sim here before the include overrides the
-       description's default of true. -->
-  <xacro:arg name="use_sim" default="false"/>
+       given name, so declaring simulator=none here before the include
+       overrides the description's default. -->
+  <xacro:arg name="simulator" default="none"/>
   <xacro:include filename="$(find base101_description)/urdf/base101.xacro"/>
   <!-- =================================================================

File: src/base101_description/urdf/base101.xacro (robot description, xacro)
@@ -2,12 +2,19 @@
 <robot name="base101" xmlns:xacro="http://www.ros.org/wiki/xacro">
   <xacro:arg name="variant" default="simple"/>
-  <!-- When true, the URDF pulls in the Gazebo ros2_control plugin and per-link
-       gazebo extensions. Hardware launches (base101_control) override to false. -->
-  <xacro:arg name="use_sim" default="true"/>
+  <!-- Which simulator the URDF is being prepared for. Selects the
+       ros2_control hardware plugin and any sim-specific extension tags.
+       Use `none` for real-hardware bringup (handled in base101_control). -->
+  <xacro:arg name="simulator" default="gazebo"/>
   <xacro:include filename="$(find base101_description)/urdf/materials.xacro"/>
   <xacro:include filename="$(find base101_description)/urdf/base101_$(arg variant).xacro"/>
-  <xacro:if value="$(arg use_sim)">
-    <xacro:include filename="$(find base101_description)/urdf/base101.ros2control"/>
+  <xacro:if value="${'$(arg simulator)' == 'gazebo'}">
+    <xacro:include filename="$(find base101_description)/urdf/base101.gazebo.ros2control"/>
     <xacro:include filename="$(find base101_description)/urdf/base101_$(arg variant).gazebo"/>
   </xacro:if>
+  <xacro:if value="${'$(arg simulator)' == 'mujoco'}">
+    <xacro:include filename="$(find base101_description)/urdf/base101.mujoco.ros2control"/>
+  </xacro:if>
+  <!-- simulator=isaac: drives joints natively from base101_isaac, no
+       ros2_control block. simulator=none: real-hardware ros2_control is
+       included from base101_control. -->
 </robot>

File: src/base101_description/urdf/base101_pro.xacro (robot description, xacro)
@@ -61,5 +61,5 @@
   </collision>
 </link>
-<link name="head_camera_1">
+<link name="base_camera">
   <inertial>
     <origin xyz="0.012450337454890298 -0.021387631051719317 -2.7969539088602835e-05" rpy="0 0 0"/>
@@ -70,5 +70,5 @@
     <origin xyz="-0.17 -0.0225 -0.043" rpy="0 0 0"/>
     <geometry>
-      <mesh filename="file://$(find base101_description)/meshes/pro/head_camera_1.stl" scale="0.001 0.001 0.001"/>
+      <mesh filename="file://$(find base101_description)/meshes/pro/base_camera.stl" scale="0.001 0.001 0.001"/>
     </geometry>
     <material name="silver"/>
@@ -77,5 +77,5 @@
     <origin xyz="-0.17 -0.0225 -0.043" rpy="0 0 0"/>
     <geometry>
-      <mesh filename="file://$(find base101_description)/meshes/pro/head_camera_1.stl" scale="0.001 0.001 0.001"/>
+      <mesh filename="file://$(find base101_description)/meshes/pro/base_camera.stl" scale="0.001 0.001 0.001"/>
     </geometry>
   </collision>
@@ -434,5 +434,5 @@
   <origin xyz="0.0 -0.0775 0.04" rpy="0 0 0"/>
   <parent link="box_front_1"/>
-  <child link="head_camera_1"/>
+  <child link="base_camera"/>
 </joint>
 <joint name="wheel_front_right" type="continuous">

File: src/base101_description/urdf/base101_simple.xacro (robot description, xacro)
@@ -62,5 +62,5 @@
   </collision>
 </link>
-<link name="head_camera_1">
+<link name="base_camera">
   <inertial>
     <origin xyz="0.012450796675630954 -0.021387754754905838 -2.7865943366574275e-05" rpy="0 0 0"/>
@@ -72,5 +72,5 @@
     <origin xyz="-0.174675 -0.014363 -0.050149" rpy="0 0 0"/>
     <geometry>
-      <mesh filename="file://$(find base101_description)/meshes/simple/head_camera_1.stl" scale="0.001 0.001 0.001"/>
+      <mesh filename="file://$(find base101_description)/meshes/simple/base_camera.stl" scale="0.001 0.001 0.001"/>
     </geometry>
     <material name="silver"/>
@@ -79,5 +79,5 @@
     <origin xyz="-0.174675 -0.014363 -0.050149" rpy="0 0 0"/>
     <geometry>
-      <mesh filename="file://$(find base101_description)/meshes/simple/head_camera_1.stl" scale="0.001 0.001 0.001"/>
+      <mesh filename="file://$(find base101_description)/meshes/simple/base_camera.stl" scale="0.001 0.001 0.001"/>
     </geometry>
   </collision>
@@ -516,5 +516,5 @@
   <origin xyz="0.0 -0.0775 0.04" rpy="0 0 0"/>
   <parent link="box_front_1"/>
-  <child link="head_camera_1"/>
+  <child link="base_camera"/>
 </joint>
 <joint name="Rigid 51" type="fixed">

Commit message: added dual arm setup

File: src/base101_control/urdf/base101.hardware.xacro (robot description, xacro)
@@ -2,4 +2,5 @@
 <robot name="base101" xmlns:xacro="http://www.ros.org/wiki/xacro">
   <xacro:arg name="variant" default="simple"/>
+  <xacro:arg name="tower" default="false"/>
   <!-- Force-disable the sim ros2_control + per-sim extensions so this URDF is
        safe to load on real hardware. Xacro takes the first <xacro:arg> for a
@@ -40,4 +41,23 @@
       <state_interface name="velocity"/>
     </joint>
+    <!-- Cross tower joints (lift column + pan/tilt head). Like the wheels,
+         mock components until the real actuator drivers land. -->
+    <xacro:if value="$(arg tower)">
+      <joint name="lift">
+        <command_interface name="position"/>
+        <state_interface name="position"/>
+        <state_interface name="velocity"/>
+      </joint>
+      <joint name="head_pan">
+        <command_interface name="position"/>
+        <state_interface name="position"/>
+        <state_interface name="velocity"/>
+      </joint>
+      <joint name="head_tilt">
+        <command_interface name="position"/>
+        <state_interface name="position"/>
+        <state_interface name="velocity"/>
+      </joint>
+    </xacro:if>
   </ros2_control>
 </robot>

File: src/base101_description/urdf/base101.xacro (robot description, xacro)
@@ -6,9 +6,24 @@
        Use `none` for real-hardware bringup (handled in base101_control). -->
   <xacro:arg name="simulator" default="gazebo"/>
+  <!-- Cross tower add-on: column with prismatic lift + pan/tilt head. -->
+  <xacro:arg name="tower" default="false"/>
+  <!-- Dual mod101 arms on the tower's crossbeam brackets. Requires
+       tower:=true and the mod101 workspace sourced as an underlay. -->
+  <xacro:arg name="arms" default="false"/>
+  <xacro:arg name="arm_tool" default="jaws"/>
   <xacro:include filename="$(find base101_description)/urdf/materials.xacro"/>
   <xacro:include filename="$(find base101_description)/urdf/base101_$(arg variant).xacro"/>
+  <xacro:if value="$(arg tower)">
+    <xacro:include filename="$(find base101_description)/urdf/base101_tower.xacro"/>
+  </xacro:if>
+  <xacro:if value="$(arg arms)">
+    <xacro:include filename="$(find base101_description)/urdf/base101_arms.xacro"/>
+  </xacro:if>
   <xacro:if value="${'$(arg simulator)' == 'gazebo'}">
     <xacro:include filename="$(find base101_description)/urdf/base101.gazebo.ros2control"/>
     <xacro:include filename="$(find base101_description)/urdf/base101_$(arg variant).gazebo"/>
+    <xacro:if value="$(arg tower)">
+      <xacro:include filename="$(find base101_description)/urdf/base101_tower.gazebo"/>
+    </xacro:if>
   </xacro:if>
   <xacro:if value="${'$(arg simulator)' == 'mujoco'}">
