Commit message: where do I even start

File: src/base101/base101_description/urdf/chassis.xacro (robot description, xacro)
@@ -1,111 +1,98 @@
 <?xml version="1.0" ?>
-<robot name="base101_simple" xmlns:xacro="http://www.ros.org/wiki/xacro">
-<!-- Pure geometry for the base101 simple variant. Materials, the gz_ros2_control
-     plugin + sensors (base101_simple.gazebo) and the ros2_control system
-     (base101.gazebo.ros2control) are pulled in by the base101.xacro dispatcher,
-     not here. The arm mount deck (hex standoffs + Component88) and the mod101
-     arm are an overlay — see the base101_arm package. -->
-<!-- base_link is recentred on the wheel-contact centroid: the raw CAD export
-     placed the origin off-centre, so the whole chassis (this link's geometry +
-     its two box children) is shifted by O = (0.0442785, 0.054181, 0) = -centroid.
-     After the shift the wheels sit symmetrically about the origin (box children
-     at Y = +/-0.12), which is what diff_drive / the nav footprint assume. -->
+<robot name="base101_chassis" xmlns:xacro="http://www.ros.org/wiki/xacro">
+<!-- Shared base101 chassis geometry. Materials, the gz_ros2_control plugin and
+     the sensor/friction extensions (chassis.gazebo, chassis.*.ros2control) are
+     pulled in by the variant xacros, not here.
+     Folded by hand from the Fusion 360 export (see scripts/import_cad_export.py
+     for the mesh side of the same import). Everything below is in the export's
+     global CAD frame, in millimetres scaled by 0.001, which is why every
+     visual/collision origin is just the negated position of its own link.
+     base_link sits on the wheel contact plane (CAD z = -81.965 mm), centred on
+     the chassis, so odom/nav/diff_drive see a ground-level origin. The rest of
+     the tree keeps the exported positions verbatim.
+     Camera choice is an argument: the edge bracket takes either a RealSense
+     D435 or a Luxonis OAK-D, and both mount to the same face. Whichever is
+     fitted, the stable frames are camera_link / camera_optical_frame. -->
+<xacro:arg name="camera" default="realsense"/>
+<!-- ================================= frame =================================
+     Two 60x20 extrusion rails plus front/back cross members, with the
+     3 mm top deck (base_link) closing the box. -->
 <link name="base_link">
   <inertial>
-    <origin xyz="-0.0009677230747272545 0.0001918701345329512 0.022138382221213098" rpy="0 0 0"/>
-    <mass value="1.8682863061101787"/>
-    <inertia ixx="0.008987" iyy="0.017929" izz="0.026913" ixy="-5e-05" iyz="0.0" ixz="0.0"/>
-  </inertial>
-  <visual>
-    <origin xyz="0.0442785 0.054181 0" rpy="0 0 0"/>
+    <origin xyz="-0.00433828 0 0.083465" rpy="0 0 0"/>
+    <mass value="1.81049"/>
+    <inertia ixx="0.00899888" iyy="0.0171197" izz="0.0261159" ixy="0" iyz="0" ixz="0"/>
+  </inertial>
+  <visual>
+    <origin xyz="0 0 0.081965" rpy="0 0 0"/>
     <geometry>
       <mesh filename="file://$(find base101_description)/meshes/base_link.stl" scale="0.001 0.001 0.001"/>
     </geometry>
-    <material name="silver"/>
-  </visual>
-  <collision>
-    <origin xyz="0.0442785 0.054181 0" rpy="0 0 0"/>
-    <geometry>
-      <mesh filename="file://$(find base101_description)/meshes/base_link.stl" scale="0.001 0.001 0.001"/>
-    </geometry>
-  </collision>
-</link>
-<link name="wheel_outside_FR_1">
-  <inertial>
-    <origin xyz="4.6650407153903117e-07 0.0032814897069334825 -3.4925017725756513e-07" rpy="0 0 0"/>
-    <mass value="0.4769861411145521"/>
-    <inertia ixx="0.000173" iyy="0.000323" izz="0.000173" ixy="-0.0" iyz="-0.0" ixz="-0.0"/>
-  </inertial>
-  <visual>
-    <origin xyz="-0.075348 0.202497 -0.037554" rpy="0 0 0"/>
-    <geometry>
-      <mesh filename="file://$(find base101_description)/meshes/wheel_outside_FR_1.stl" scale="0.001 0.001 0.001"/>
-    </geometry>
-    <material name="silver"/>
-  </visual>
-  <collision>
-    <origin xyz="-0.075348 0.202497 -0.037554" rpy="0 0 0"/>
-    <geometry>
-      <mesh filename="file://$(find base101_description)/meshes/wheel_outside_FR_1.stl" scale="0.001 0.001 0.001"/>
-    </geometry>
-  </collision>
-</link>
-<link name="wheel_outside_FL_1">
-  <inertial>
-    <origin xyz="4.5391676331552056e-07 -0.0032816238538548592 4.0204846763619573e-07" rpy="0 0 0"/>
-    <mass value="0.4769861411145521"/>
-    <inertia ixx="0.000173" iyy="0.000323" izz="0.000173" ixy="0.0" iyz="-0.0" ixz="-0.0"/>
-  </inertial>
-  <visual>
-    <origin xyz="-0.075348 -0.094135 -0.037671" rpy="0 0 0"/>
-    <geometry>
-      <mesh filename="file://$(find base101_description)/meshes/wheel_outside_FL_1.stl" scale="0.001 0.001 0.001"/>
-    </geometry>
-    <material name="silver"/>
-  </visual>
-  <collision>
-    <origin xyz="-0.075348 -0.094135 -0.037671" rpy="0 0 0"/>
-    <geometry>
-      <mesh filename="file://$(find base101_description)/meshes/wheel_outside_FL_1.stl" scale="0.001 0.001 0.001"/>
-    </geometry>
-  </collision>
-</link>
-<link name="wheel_outside_BL_1">
-  <inertial>
-    <origin xyz="1.060114172835025e-07 -0.0032816238538547204 4.263746731583695e-07" rpy="0 0 0"/>
-    <mass value="0.4769861411145521"/>
-    <inertia ixx="0.000173" iyy="0.000323" izz="0.000173" ixy="0.0" iyz="-0.0" ixz="0.0"/>
-  </inertial>
-  <visual>
-    <origin xyz="0.163905 -0.094135 -0.037671" rpy="0 0 0"/>
-    <geometry>
-      <mesh filename="file://$(find base101_description)/meshes/wheel_outside_BL_1.stl" scale="0.001 0.001 0.001"/>
-    </geometry>
-    <material name="silver"/>
-  </visual>
-  <collision>
-    <origin xyz="0.163905 -0.094135 -0.037671" rpy="0 0 0"/>
-    <geometry>
-      <mesh filename="file://$(find base101_description)/meshes/wheel_outside_BL_1.stl" scale="0.001 0.001 0.001"/>
-    </geometry>
-  </collision>
-</link>
-<link name="wheel_outside_BR_1">
-  <inertial>
-    <origin xyz="6.387720691281018e-08 0.003281489706936147 -3.9622663744465214e-07" rpy="0 0 0"/>
-    <mass value="0.4769861411145521"/>
-    <inertia ixx="0.000173" iyy="0.000323" izz="0.000173" ixy="0.0" iyz="0.0" ixz="0.0"/>
-  </inertial>
-  <visual>
-    <origin xyz="0.163905 0.202497 -0.037554" rpy="0 0 0"/>
-    <geometry>
-      <mesh filename="file://$(find base101_description)/meshes/wheel_outside_BR_1.stl" scale="0.001 0.001 0.001"/>
-    </geometry>
-    <material name="silver"/>
-  </visual>
-  <collision>
-    <origin xyz="0.163905 0.202497 -0.037554" rpy="0 0 0"/>
-    <geometry>
-      <mesh filename="file://$(find base101_description)/meshes/wheel_outside_BR_1.stl" scale="0.001 0.001 0.001"/>
+    <material name="plate_aluminum"/>
+  </visual>
+  <collision>
+    <origin xyz="0 0 0.083465" rpy="0 0 0"/>
+    <geometry>
+      <box size="0.34 0.24 0.003"/>
+    </geometry>
+  </collision>
+</link>
+<link name="box_front_1">
+  <inertial>
+    <origin xyz="-0.00962595 0 -0.03" rpy="0 0 0"/>
+    <mass value="0.740521"/>
+    <inertia ixx="0.003275" iyy="0.000289" izz="0.003048" ixy="0" iyz="0" ixz="0"/>
+  </inertial>
+  <visual>
+    <origin xyz="-0.17 0 0" rpy="0 0 0"/>
+    <geometry>
+      <mesh filename="file://$(find base101_description)/meshes/box_front_1.stl" scale="0.001 0.001 0.001"/>
+    </geometry>
+    <material name="extrusion_grey"/>
+  </visual>
+  <collision>
+    <origin xyz="-0.01 0 -0.03" rpy="0 0 0"/>
+    <geometry>
+      <box size="0.02 0.24 0.06"/>
+    </geometry>
+  </collision>
+</link>
+<link name="box_back_1">
+  <inertial>
+    <origin xyz="0.00962595 0 -0.03" rpy="0 0 0"/>
+    <mass value="0.740521"/>
+    <inertia ixx="0.003275" iyy="0.000289" izz="0.003048" ixy="0" iyz="0" ixz="0"/>
+  </inertial>
+  <visual>
+    <origin xyz="0.17 0 0" rpy="0 0 0"/>
+    <geometry>
+      <mesh filename="file://$(find base101_description)/meshes/box_back_1.stl" scale="0.001 0.001 0.001"/>
+    </geometry>
+    <material name="extrusion_grey"/>
+  </visual>
+  <collision>
+    <origin xyz="0.01 0 -0.03" rpy="0 0 0"/>
+    <geometry>
+      <box size="0.02 0.24 0.06"/>
+    </geometry>
+  </collision>
+</link>
+<link name="box_left_1">
+  <inertial>
+    <origin xyz="-0.17 -0.00974265 -0.0299929" rpy="0 0 0"/>
+    <mass value="1.07632"/>
+    <inertia ixx="0.00042" iyy="0.009599" izz="0.009268" ixy="0" iyz="0" ixz="0"/>
+  </inertial>
+  <visual>
+    <origin xyz="-0.17 -0.12 0" rpy="0 0 0"/>
+    <geometry>
+      <mesh filename="file://$(find base101_description)/meshes/box_left_1.stl" scale="0.001 0.001 0.001"/>
+    </geometry>
+    <material name="extrusion_grey"/>
+  </visual>
+  <collision>
+    <origin xyz="-0.17 -0.01 -0.03" rpy="0 0 0"/>
+    <geometry>
+      <box size="0.34 0.02 0.06"/>
     </geometry>
   </collision>
@@ -113,219 +100,580 @@
 <link name="box_right_1">
   <inertial>
-    <origin xyz="-0.1699997988923434 0.009999932926543414 0.03000707550989725" rpy="0 0 0"/>
-    <mass value="1.143643042060448"/>
-    <inertia ixx="0.000446" iyy="0.011412" izz="0.01106" ixy="-0.0" iyz="-0.0" ixz="0.0"/>
-  </inertial>
-  <visual>
-    <origin xyz="-0.125291 0.174181 -0.023638" rpy="0 0 0"/>
+    <origin xyz="-0.17 0.00974265 -0.0299929" rpy="0 0 0"/>
+    <mass value="1.07632"/>
+    <inertia ixx="0.00042" iyy="0.009599" izz="0.009268" ixy="0" iyz="0" ixz="0"/>
+  </inertial>
+  <visual>
+    <origin xyz="-0.17 0.12 0" rpy="0 0 0"/>
     <geometry>
       <mesh filename="file://$(find base101_description)/meshes/box_right_1.stl" scale="0.001 0.001 0.001"/>
     </geometry>
-    <material name="silver"/>
-  </visual>
-  <collision>
-    <origin xyz="-0.125291 0.174181 -0.023638" rpy="0 0 0"/>
-    <geometry>
-      <mesh filename="file://$(find base101_description)/meshes/box_right_1.stl" scale="0.001 0.001 0.001"/>
-    </geometry>
-  </collision>
-</link>
-<link name="box_left_1">
-  <inertial>
-    <origin xyz="-0.16999979889234568 -0.010000067073461412 0.030007075509897126" rpy="0 0 0"/>
-    <mass value="1.143643042060435"/>
-    <inertia ixx="0.000446" iyy="0.011412" izz="0.01106" ixy="-0.0" iyz="-0.0" ixz="0.0"/>
-  </inertial>
-  <visual>
-    <origin xyz="-0.125291 -0.065819 -0.023638" rpy="0 0 0"/>
-    <geometry>
-      <mesh filename="file://$(find base101_description)/meshes/box_left_1.stl" scale="0.001 0.001 0.001"/>
-    </geometry>
-    <material name="silver"/>
-  </visual>
-  <collision>
-    <origin xyz="-0.125291 -0.065819 -0.023638" rpy="0 0 0"/>
-    <geometry>
-      <mesh filename="file://$(find base101_description)/meshes/box_left_1.stl" scale="0.001 0.001 0.001"/>
-    </geometry>
-  </collision>
-</link>
-<link name="box_front_1">
-  <inertial>
-    <origin xyz="-0.009999798892348241 -0.10000006707345671 0.029994444121839027" rpy="0 0 0"/>
-    <mass value="0.6728017040951292"/>
-    <inertia ixx="0.002479" iyy="0.000262" izz="0.002271" ixy="-0.0" iyz="0.0" ixz="0.0"/>
-  </inertial>
-  <visual>
-    <origin xyz="-0.125291 -0.045819 -0.023638" rpy="0 0 0"/>
-    <geometry>
-      <mesh filename="file://$(find base101_description)/meshes/box_front_1.stl" scale="0.001 0.001 0.001"/>
-    </geometry>
-    <material name="silver"/>
-  </visual>
-  <collision>
-    <origin xyz="-0.125291 -0.045819 -0.023638" rpy="0 0 0"/>
-    <geometry>
-      <mesh filename="file://$(find base101_description)/meshes/box_front_1.stl" scale="0.001 0.001 0.001"/>
-    </geometry>
-  </collision>
-</link>
-<link name="box_back_1">
-  <inertial>
-    <origin xyz="0.010000201107653484 -0.10000006707346183 0.0300003822212132" rpy="0 0 0"/>
-    <mass value="0.673201220432864"/>
-    <inertia ixx="0.002479" iyy="0.000262" izz="0.002272" ixy="-0.0" iyz="-0.0" ixz="0.0"/>
-  </inertial>
-  <visual>
-    <origin xyz="0.214709 -0.045819 -0.023638" rpy="0 0 0"/>
-    <geometry>
-      <mesh filename="file://$(find base101_description)/meshes/box_back_1.stl" scale="0.001 0.001 0.001"/>
-    </geometry>
-    <material name="silver"/>
-  </visual>
-  <collision>
-    <origin xyz="0.214709 -0.045819 -0.023638" rpy="0 0 0"/>
-    <geometry>
-      <mesh filename="file://$(find base101_description)/meshes/box_back_1.stl" scale="0.001 0.001 0.001"/>
-    </geometry>
-  </collision>
-</link>
-<link name="imu_1">
-  <inertial>
-    <origin xyz="0.007620201107655988 -0.010160067073459976 -0.0007996177787881475" rpy="0 0 0"/>
-    <mass value="0.0060600570697449205"/>
-    <inertia ixx="0.0" iyy="0.0" izz="0.0" ixy="-0.0" iyz="0.0" ixz="0.0"/>
-  </inertial>
-  <visual>
-    <origin xyz="0.107459 0.044081 -0.077138" rpy="0 0 0"/>
-    <geometry>
-      <mesh filename="file://$(find base101_description)/meshes/imu_1.stl" scale="0.001 0.001 0.001"/>
-    </geometry>
-    <material name="silver"/>
-  </visual>
-  <collision>
-    <origin xyz="0.107459 0.044081 -0.077138" rpy="0 0 0"/>
-    <geometry>
-      <mesh filename="file://$(find base101_description)/meshes/imu_1.stl" scale="0.001 0.001 0.001"/>
-    </geometry>
-  </collision>
-</link>
-<link name="connector_mask_1">
-  <inertial>
-    <origin xyz="-1.337822052970403 1.7039662491302847 -1.079899943041819" rpy="0 0 0"/>
-    <mass value="0.14432039780190548"/>
-    <inertia ixx="6.8e-05" iyy="2e-05" izz="8.7e-05" ixy="0.0" iyz="0.0" ixz="0.0"/>
-  </inertial>
-  <visual>
-    <origin xyz="-1.241617 1.758011 -1.162022" rpy="0 0 0"/>
-    <geometry>
-      <mesh filename="file://$(find base101_description)/meshes/connector_mask_1.stl" scale="0.001 0.001 0.001"/>
-    </geometry>
-    <material name="silver"/>
-  </visual>
-  <collision>
-    <origin xyz="-1.241617 1.758011 -1.162022" rpy="0 0 0"/>
-    <geometry>
-      <mesh filename="file://$(find base101_description)/meshes/connector_mask_1.stl" scale="0.001 0.001 0.001"/>
-    </geometry>
-  </collision>
-</link>
-<link name="baseus_1">
-  <inertial>
-    <origin xyz="0.07757535171107266 -6.707346256185076e-08 -0.026277531510434472" rpy="0 0 0"/>
-    <mass value="2.7975020361255334"/>
-    <inertia ixx="0.001064" iyy="0.006218" izz="0.006047" ixy="-0.0" iyz="0.0" ixz="-1.4e-05"/>
-  </inertial>
-  <visual>
-    <origin xyz="0.182114 0.124481 -0.08066" rpy="0 0 0"/>
-    <geometry>
-      <mesh filename="file://$(find base101_description)/meshes/baseus_1.stl" scale="0.001 0.001 0.001"/>
-    </geometry>
-    <material name="silver"/>
-  </visual>
-  <collision>
-    <origin xyz="0.182114 0.124481 -0.08066" rpy="0 0 0"/>
-    <geometry>
-      <mesh filename="file://$(find base101_description)/meshes/baseus_1.stl" scale="0.001 0.001 0.001"/>
-    </geometry>
-  </collision>
-</link>
-<link name="baseus_back_holder_1">
-  <inertial>
-    <origin xyz="0.0018606296791154053 0.0196913856625118 -0.023384735966532046" rpy="0 0 0"/>
-    <mass value="0.06553080969569097"/>
-    <inertia ixx="5.4e-05" iyy="3.1e-05" izz="2.4e-05" ixy="-0.0" iyz="0.0" ixz="1e-06"/>
-  </inertial>
-  <visual>
-    <origin xyz="0.184709 0.144181 -0.083638" rpy="0 0 0"/>
-    <geometry>
-      <mesh filename="file://$(find base101_description)/meshes/baseus_back_holder_1.stl" scale="0.001 0.001 0.001"/>
-    </geometry>
-    <material name="silver"/>
-  </visual>
-  <collision>
-    <origin xyz="0.184709 0.144181 -0.083638" rpy="0 0 0"/>
-    <geometry>
-      <mesh filename="file://$(find base101_description)/meshes/baseus_back_holder_1.stl" scale="0.001 0.001 0.001"/>
-    </geometry>
-  </collision>
-</link>
-<link name="connector_cap_r_1">
-  <inertial>
-    <origin xyz="0.015000201107883693 -6.707345745482485e-08 0.0029246117479597156" rpy="0 0 0"/>
-    <mass value="0.03612758231947257"/>
-    <inertia ixx="2e-06" iyy="9e-06" izz="1e-05" ixy="0.0" iyz="-0.0" ixz="0.0"/>
-  </inertial>
-  <visual>
-    <origin xyz="0.094709 0.144181 -0.083638" rpy="0 0 0"/>
-    <geometry>
-      <mesh filename="file://$(find base101_description)/meshes/connector_cap_r_1.stl" scale="0.001 0.001 0.001"/>
-    </geometry>
-    <material name="silver"/>
-  </visual>
-  <collision>
-    <origin xyz="0.094709 0.144181 -0.083638" rpy="0 0 0"/>
-    <geometry>
-      <mesh filename="file://$(find base101_description)/meshes/connector_cap_r_1.stl" scale="0.001 0.001 0.001"/>
-    </geometry>
-  </collision>
-</link>
-<link name="baseus_front_holder_1">
-  <inertial>
-    <origin xyz="-0.0018602281494875736 0.019691385658470797 -0.023384741531271826" rpy="0 0 0"/>
-    <mass value="0.06553077927945053"/>
-    <inertia ixx="5.4e-05" iyy="3.1e-05" izz="2.4e-05" ixy="0.0" iyz="0.0" ixz="-1e-06"/>
-  </inertial>
-  <visual>
-    <origin xyz="0.024709 0.144181 -0.083638" rpy="0 0 0"/>
-    <geometry>
-      <mesh filename="file://$(find base101_description)/meshes/baseus_front_holder_1.stl" scale="0.001 0.001 0.001"/>
-    </geometry>
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
File: src/base101/base101_description/urdf/materials.xacro (robot description, xacro)
@@ -1,4 +1,37 @@
 <?xml version="1.0" ?>
 <robot name="base101" xmlns:xacro="http://www.ros.org/wiki/xacro">
+  <!-- Palette is by material, not by part, so a new link picks its colour from
+       what it is made of. Gazebo equivalents are in chassis.gazebo and must be
+       kept in step. -->
+  <!-- 60x20 extrusion, black anodized: reads dark grey under light. -->
+  <material name="extrusion_grey">
+    <color rgba="0.220 0.225 0.235 1.0"/>
+  </material>
+  <!-- 3 mm CNC aluminium: the base deck and the payload plate. -->
+  <material name="plate_aluminum">
+    <color rgba="0.770 0.780 0.790 1.0"/>
+  </material>
+  <!-- Everything printed: PLA-CF mounts and brackets, TPU bumpers. -->
+  <material name="plastic_black">
+    <color rgba="0.075 0.075 0.080 1.0"/>
+  </material>
+  <!-- Standoffs and fasteners. -->
+  <material name="hardware_steel">
+    <color rgba="0.600 0.605 0.620 1.0"/>
+  </material>
+  <!-- Bare PCB (the link101 carrier board). -->
+  <material name="pcb_green">
+    <color rgba="0.055 0.260 0.140 1.0"/>
+  </material>
+  <!-- Anodised/moulded electronics housings: cameras, the Orin. -->
+  <material name="electronics_grey">
+    <color rgba="0.300 0.310 0.330 1.0"/>
+  </material>
+  <!-- DDSM210 hub motors and the lidar can. -->
+  <material name="motor_black">
+    <color rgba="0.050 0.050 0.050 1.0"/>
+  </material>
+  <!-- Kept for the add-on packages (base101_arm, the parked tower) and the
+       mod101 macro, which reference these names directly. -->
   <material name="silver">
     <color rgba="0.700 0.700 0.700 1.0"/>
@@ -10,6 +43,3 @@
     <color rgba="0.180 0.580 0.270 1.0"/>
   </material>
-  <material name="motor_black">
-    <color rgba="0.050 0.050 0.050 1.0"/>
-  </material>
 </robot>

File: src/base101/base101_simple_description/urdf/base101_simple.xacro (robot description, xacro)
@@ -9,4 +9,8 @@
        ros2_control or extension tags). -->
   <xacro:arg name="simulator" default="gazebo"/>
+  <!-- Which module is on the front bracket: realsense | oak_d. Declared by
+       chassis.xacro too; repeated here so the variant's own argument list is
+       complete and it can be overridden per launch. -->
+  <xacro:arg name="camera" default="realsense"/>
   <!-- Shared chassis: chassis links + materials. -->
   <xacro:include filename="$(find base101_description)/urdf/materials.xacro"/>

File: src/base101_arm/base101_arm_description/urdf/arm.xacro (robot description, xacro)
@@ -1,10 +1,22 @@
 <?xml version="1.0" ?>
 <robot name="base101_arm" xmlns:xacro="http://www.ros.org/wiki/xacro">
-<!-- One mod101 arm on the arm mount plate. Included from base101_arm.xacro
-     when arm:=true. mod101 stays a standalone repo: build it first and source
-     its install as an underlay, then build this workspace.
-     Joint names become arm_1..arm_6; controllers live in
+<!-- One mod101 arm on the chassis deck. Included from base101_arm.xacro when
+     arm:=true. mod101 stays a standalone repo: build it first and source its
+     install as an underlay, then build this workspace.
+     Joint names get the arm_ prefix (arm_joint_base ... arm_joint_wrist_roll,
+     plus the tool's arm_6); controllers live in
      base101_arm_control/config/controllers.sim.yaml. -->
+<!-- How the arm is built is the web configurator's call, not ours. Including
+     mod101_config.xacro gives us the same tool + rail lengths + servo mounts
+     the configurator last wrote, so re-running it and rebuilding is enough to
+     change the arm here. Passing these explicitly matters: leave any of them
+     off and the macro silently falls back to its own signature defaults, which
+     are NOT the configured values. -->
+<xacro:include filename="$(find mod101_description)/urdf/mod101_config.xacro"/>
 <xacro:include filename="$(find mod101_description)/urdf/mod101_macro.xacro"/>
+<!-- Tool follows the configurator too, but stays overridable per launch
+     (arm_tool:=parallel) so you can run a different end-effector on the robot
+     than on the bench. -->
+<xacro:arg name="arm_tool" default="$(arg tool)"/>
 <!-- The only mod101 material base101's palette doesn't already define
      (silver / accent_green / motor_black match byte-for-byte). -->
@@ -15,11 +27,16 @@
      mujoco scenes don't model it yet and simulator=none is rviz-only. -->
 <xacro:property name="arm_use_sim" value="${'$(arg simulator)' == 'gazebo'}"/>
-<!-- Mount point on the arm mount plate top face: the plate is ~160x220 mm and
-     its top deck sits ~3 mm above the link origin; the arm base (80x100 mm)
-     drops onto the plate centre (the plate's own inertial centroid in XY).
-     Refine against the physical bolt pattern. Unrotated, the arm's ready
-     stance reaches toward the robot's front (+X). -->
-<xacro:mod101_arm prefix="arm_" parent="arm_mount_plate"
-                  xyz="-0.08 0.11 0.01" rpy="0 0 0"
-                  tool="$(arg arm_tool)" use_sim="${arm_use_sim}"/>
+<!-- Mount point on the chassis deck (top_plate_1) top face. mod101's
+     base_link sits at the centre of its own base plate on the mounting face,
+     so this is just "deck centre, deck top" in deck-local coords: the deck
+     origin is its back-right corner (base_link -0.08, -0.11), 3 mm under the
+     top face.
+     Unrotated, the arm's ready stance reaches toward the robot's front (+X). -->
+<xacro:mod101_arm prefix="arm_" parent="top_plate_1"
+                  xyz="0.08 0.11 0.003" rpy="0 0 0"
+                  tool="$(arg arm_tool)" use_sim="${arm_use_sim}"
+                  shoulder_ext_length="$(arg shoulder_ext_length)"
+                  elbow_ext_length="$(arg elbow_ext_length)"
+                  shoulder_mount="$(arg shoulder_mount)"
+                  elbow_mount="$(arg elbow_mount)"/>
 </robot>
