Commit message: where do I even start

File: src/base101_arm/base101_arm_description/urdf/base101_arm.xacro (robot description, xacro)
@@ -1,6 +1,9 @@
 <?xml version="1.0" ?>
 <!-- base101 "arm" variant: chassis + a single deck-mounted mod101 arm.
-     Assembles the shared chassis (base101_description) and layers the arm
-     mount deck (hex standoffs + arm_mount_plate) and one mod101 arm on top.
+     Assembles the shared chassis (base101_description) and puts one mod101
+     arm on its deck. There is no mount deck of its own any more: the 2026-08
+     chassis re-export raised top_plate_1 onto 45 mm standoffs, which is
+     exactly what this package used to add on top of the old flat deck, so the
+     arm bolts straight to the chassis.
      `arm:=true` requires the mod101 underlay sourced (build mod101 first).
      Controllers live in base101_arm_control. -->
@@ -8,11 +11,10 @@
   <xacro:arg name="simulator" default="gazebo"/>
   <xacro:arg name="arm" default="true"/>
-  <xacro:arg name="arm_tool" default="jaws"/>
+  <!-- arm_tool is declared in arm.xacro, defaulting to the configurator's
+       `tool`. Declaring it here with a literal default would shadow that. -->
   <!-- Shared chassis. -->
   <xacro:include filename="$(find base101_description)/urdf/materials.xacro"/>
   <xacro:include filename="$(find base101_description)/urdf/chassis.xacro"/>
-  <!-- Arm mount deck (hex standoffs + arm_mount_plate) onto top_plate_1. -->
-  <xacro:include filename="$(find base101_arm_description)/urdf/arm_mount.xacro"/>
-  <!-- One mod101 arm on the arm_mount_plate. -->
+  <!-- One mod101 arm on the chassis deck. -->
   <xacro:if value="$(arg arm)">
     <xacro:include filename="$(find base101_arm_description)/urdf/arm.xacro"/>
@@ -21,5 +23,4 @@
     <xacro:include filename="$(find base101_description)/urdf/chassis.gazebo.ros2control"/>
     <xacro:include filename="$(find base101_description)/urdf/chassis.gazebo"/>
-    <xacro:include filename="$(find base101_arm_description)/urdf/arm_mount.gazebo"/>
     <!-- gz_ros2_control loads this variant's controllers (wheels + arm). The
          arm joints' ros2_control blocks are emitted by the mod101 macro

Commit message: changed bumpers, integrated moveit, nicer readme

File: src/base101/base101_description/urdf/chassis.xacro (robot description, xacro)
@@ -424,5 +424,23 @@
 </joint>
 <!-- ================================ bumpers ================================
-     TPU corner pieces, press-fit onto the extrusion ends. -->
+     TPU corner pieces, press-fit onto the extrusion ends.
+     2026-08 revision: rounded cosmetic redesign. The press-fit body is
+     UNCHANGED at 60 x 60 x 66 mm and still sits on the extrusion at |x|=130,
+     |y|=80 mm. What is new is two 12 mm fins (at z=-20..-8 and -52..-40 in CAD)
+     that protrude 5 mm further out, so the envelope grows 380 x 280 ->
+     390 x 290 mm. The top plate is shorter than the bumpers in X, so the
+     bumpers set the footprint in both axes.
+     IMPORTING A NEW EXPORT — three things bit us, in order:
+       1. bumper_assembly.stl holds THREE disconnected bodies (main + 2 fins),
+          not one. Treat them as one part but datum on the MAIN body, not on
+          the whole-assembly bounding box, or the fins pull the datum 5 mm off.
+       2. The export is the FRONT-RIGHT corner: its fins protrude +X and -Y.
+          For a target quadrant (qx, qy) the mirror is (qx, -qy).
+       3. The export's absolute XY is arbitrary (Z happens to be right), so
+          datum the main body's inner faces to |x|=130, |y|=80 rather than
+          trusting the exported position.
+     Only one corner is exported; the other three are mirrors, as before.
+     Collision stays a box primitive, not the mesh: the part is rounded with no
+     flat faces, and a 65 mm box covering body+fins is cheap and conservative. -->
 <link name="bumper_front_left_1">
   <inertial>
@@ -439,7 +457,7 @@
   </visual>
   <collision>
-    <origin xyz="-0.01 -0.01 -0.033" rpy="0 0 0"/>
-    <geometry>
-      <box size="0.06 0.06 0.066"/>
+    <origin xyz="-0.0075 -0.0075 -0.033" rpy="0 0 0"/>
+    <geometry>
+      <box size="0.065 0.065 0.066"/>
     </geometry>
   </collision>
@@ -459,7 +477,7 @@
   </visual>
   <collision>
-    <origin xyz="-0.01 0.01 -0.033" rpy="0 0 0"/>
-    <geometry>
-      <box size="0.06 0.06 0.066"/>
+    <origin xyz="-0.0075 0.0075 -0.033" rpy="0 0 0"/>
+    <geometry>
+      <box size="0.065 0.065 0.066"/>
     </geometry>
   </collision>
@@ -479,7 +497,7 @@
   </visual>
   <collision>
-    <origin xyz="0.01 -0.01 -0.033" rpy="0 0 0"/>
-    <geometry>
-      <box size="0.06 0.06 0.066"/>
+    <origin xyz="0.0075 -0.0075 -0.033" rpy="0 0 0"/>
+    <geometry>
+      <box size="0.065 0.065 0.066"/>
     </geometry>
   </collision>
@@ -499,7 +517,7 @@
   </visual>
   <collision>
-    <origin xyz="0.01 0.01 -0.033" rpy="0 0 0"/>
-    <geometry>
-      <box size="0.06 0.06 0.066"/>
+    <origin xyz="0.0075 0.0075 -0.033" rpy="0 0 0"/>
+    <geometry>
+      <box size="0.065 0.065 0.066"/>
     </geometry>
   </collision>
@@ -718,5 +736,9 @@
      One bracket, two options. camera_link is the front face of whichever
      module is fitted, +X out of the lens; camera_optical_frame is the
-     REP-103 optical twist of it for point clouds. -->
+     REP-103 optical twist of it (z out of the lens, x right, y down).
+     camera_optical_frame is what image and camera_info messages are stamped
+     with — matching realsense2_camera and depthai, so the frame graph does not
+     change when the real module replaces the sim one. camera_link stays the
+     mount point you position in CAD. See docs/robocore-camera-frames.md. -->
 <link name="camera_edge_bracket_1">
   <inertial>

File: src/base101_arm/base101_arm_moveit_config/config/collisions/jaws.srdf.xacro (robot description, xacro)
@@ -3,8 +3,8 @@
   GENERATED by base101_arm_moveit_config/scripts/gen_collision_matrix.py
   — do not edit by hand.
-  tool=jaws  shoulder_ext_length=0.1400 elbow_ext_length=0.1400 shoulder_mount=small elbow_mount=small
-  855 chassis-involving pairs disabled (54 adjacent/always,
-  797 never-colliding over 1000000 random samples, 4 rigid/
-  collapsed-adjacent from URDF topology), out of 1830 pairs in the
+  tool=jaws  shoulder_ext_length=0.2400 elbow_ext_length=0.2800 shoulder_mount=small elbow_mount=small
+  835 chassis-involving pairs disabled (54 adjacent/always,
+  777 never-colliding over 1000000 random samples, 4 rigid/
+  collapsed-adjacent from URDF topology), out of 1891 pairs in the
   composed robot. "Never" is statistical — see the generator's docstring for
   the trials-vs-pairs convergence on this robot. The rigid/collapsed pairs are
@@ -117,8 +117,6 @@
   <disable_collisions link1="arm_camera_adapter_1" link2="bumper_back_left_1" reason="Never"/>
   <disable_collisions link1="arm_camera_adapter_1" link2="bumper_back_right_1" reason="Never"/>
-  <disable_collisions link1="arm_camera_adapter_1" link2="jetson_mount_1" reason="Never"/>
   <disable_collisions link1="arm_camera_adapter_1" link2="mount_back_left_1" reason="Never"/>
   <disable_collisions link1="arm_camera_adapter_1" link2="mount_back_right_1" reason="Never"/>
-  <disable_collisions link1="arm_camera_adapter_1" link2="orin_simplified_1" reason="Never"/>
   <disable_collisions link1="arm_camera_adapter_1" link2="standoff_back_left_1" reason="Never"/>
   <disable_collisions link1="arm_camera_adapter_1" link2="standoff_back_right_1" reason="Never"/>
@@ -128,8 +126,6 @@
   <disable_collisions link1="arm_camera_wing_1" link2="bumper_back_left_1" reason="Never"/>
   <disable_collisions link1="arm_camera_wing_1" link2="bumper_back_right_1" reason="Never"/>
-  <disable_collisions link1="arm_camera_wing_1" link2="jetson_mount_1" reason="Never"/>
   <disable_collisions link1="arm_camera_wing_1" link2="mount_back_left_1" reason="Never"/>
   <disable_collisions link1="arm_camera_wing_1" link2="mount_back_right_1" reason="Never"/>
-  <disable_collisions link1="arm_camera_wing_1" link2="orin_simplified_1" reason="Never"/>
   <disable_collisions link1="arm_camera_wing_1" link2="standoff_back_left_1" reason="Never"/>
   <disable_collisions link1="arm_camera_wing_1" link2="standoff_back_right_1" reason="Never"/>
@@ -200,33 +196,21 @@
   <disable_collisions link1="arm_forearm_extrusion_1" link2="bumper_back_right_1" reason="Never"/>
   <disable_collisions link1="arm_forearm_extrusion_1" link2="jetson_mount_1" reason="Never"/>
-  <disable_collisions link1="arm_forearm_extrusion_1" link2="link_101_1" reason="Never"/>
   <disable_collisions link1="arm_forearm_extrusion_1" link2="mount_back_left_1" reason="Never"/>
   <disable_collisions link1="arm_forearm_extrusion_1" link2="mount_back_right_1" reason="Never"/>
   <disable_collisions link1="arm_forearm_extrusion_1" link2="orin_simplified_1" reason="Never"/>
-  <disable_collisions link1="arm_forearm_extrusion_1" link2="orp_link101_mount_1" reason="Never"/>
   <disable_collisions link1="arm_forearm_extrusion_1" link2="standoff_back_left_1" reason="Never"/>
   <disable_collisions link1="arm_forearm_extrusion_1" link2="standoff_back_right_1" reason="Never"/>
   <disable_collisions link1="arm_forearm_extrusion_1" link2="wheel_back_left_1" reason="Never"/>
   <disable_collisions link1="arm_forearm_extrusion_1" link2="wheel_back_right_1" reason="Never"/>
-  <disable_collisions link1="arm_jaws_body" link2="box_back_1" reason="Never"/>
-  <disable_collisions link1="arm_jaws_body" link2="bumper_back_left_1" reason="Never"/>
-  <disable_collisions link1="arm_jaws_body" link2="bumper_back_right_1" reason="Never"/>
   <disable_collisions link1="arm_jaws_body" link2="mount_back_left_1" reason="Never"/>
   <disable_collisions link1="arm_jaws_body" link2="mount_back_right_1" reason="Never"/>
-  <disable_collisions link1="arm_jaws_body" link2="standoff_back_left_1" reason="Never"/>
-  <disable_collisions link1="arm_jaws_body" link2="standoff_back_right_1" reason="Never"/>
   <disable_collisions link1="arm_jaws_body" link2="wheel_back_left_1" reason="Never"/>
   <disable_collisions link1="arm_jaws_body" link2="wheel_back_right_1" reason="Never"/>
-  <disable_collisions link1="arm_jaws_moving" link2="box_back_1" reason="Never"/>
-  <disable_collisions link1="arm_jaws_moving" link2="bumper_back_left_1" reason="Never"/>
-  <disable_collisions link1="arm_jaws_moving" link2="bumper_back_right_1" reason="Never"/>
   <disable_collisions link1="arm_jaws_moving" link2="mount_back_left_1" reason="Never"/>
   <disable_collisions link1="arm_jaws_servo" link2="box_back_1" reason="Never"/>
   <disable_collisions link1="arm_jaws_servo" link2="bumper_back_left_1" reason="Never"/>
   <disable_collisions link1="arm_jaws_servo" link2="bumper_back_right_1" reason="Never"/>
-  <disable_collisions link1="arm_jaws_servo" link2="jetson_mount_1" reason="Never"/>
   <disable_collisions link1="arm_jaws_servo" link2="mount_back_left_1" reason="Never"/>
   <disable_collisions link1="arm_jaws_servo" link2="mount_back_right_1" reason="Never"/>
-  <disable_collisions link1="arm_jaws_servo" link2="orin_simplified_1" reason="Never"/>
   <disable_collisions link1="arm_jaws_servo" link2="standoff_back_left_1" reason="Never"/>
   <disable_collisions link1="arm_jaws_servo" link2="standoff_back_right_1" reason="Never"/>
@@ -408,8 +392,6 @@
   <disable_collisions link1="arm_wrist_camera_v1_1" link2="bumper_back_left_1" reason="Never"/>
   <disable_collisions link1="arm_wrist_camera_v1_1" link2="bumper_back_right_1" reason="Never"/>
-  <disable_collisions link1="arm_wrist_camera_v1_1" link2="jetson_mount_1" reason="Never"/>
   <disable_collisions link1="arm_wrist_camera_v1_1" link2="mount_back_left_1" reason="Never"/>
   <disable_collisions link1="arm_wrist_camera_v1_1" link2="mount_back_right_1" reason="Never"/>
-  <disable_collisions link1="arm_wrist_camera_v1_1" link2="orin_simplified_1" reason="Never"/>
   <disable_collisions link1="arm_wrist_camera_v1_1" link2="standoff_back_left_1" reason="Never"/>
   <disable_collisions link1="arm_wrist_camera_v1_1" link2="standoff_back_right_1" reason="Never"/>
@@ -431,9 +413,7 @@
   <disable_collisions link1="arm_wrist_servo_adapter_1" link2="bumper_back_right_1" reason="Never"/>
   <disable_collisions link1="arm_wrist_servo_adapter_1" link2="jetson_mount_1" reason="Never"/>
-  <disable_collisions link1="arm_wrist_servo_adapter_1" link2="link_101_1" reason="Never"/>
   <disable_collisions link1="arm_wrist_servo_adapter_1" link2="mount_back_left_1" reason="Never"/>
   <disable_collisions link1="arm_wrist_servo_adapter_1" link2="mount_back_right_1" reason="Never"/>
   <disable_collisions link1="arm_wrist_servo_adapter_1" link2="orin_simplified_1" reason="Never"/>
-  <disable_collisions link1="arm_wrist_servo_adapter_1" link2="orp_link101_mount_1" reason="Never"/>
   <disable_collisions link1="arm_wrist_servo_adapter_1" link2="standoff_back_left_1" reason="Never"/>
   <disable_collisions link1="arm_wrist_servo_adapter_1" link2="standoff_back_right_1" reason="Never"/>

File: src/base101_arm/base101_arm_moveit_config/config/collisions/none.srdf.xacro (robot description, xacro)
@@ -3,8 +3,8 @@
   GENERATED by base101_arm_moveit_config/scripts/gen_collision_matrix.py
   — do not edit by hand.
-  tool=none  shoulder_ext_length=0.1400 elbow_ext_length=0.1400 shoulder_mount=small elbow_mount=small
-  842 chassis-involving pairs disabled (54 adjacent/always,
-  784 never-colliding over 1000000 random samples, 4 rigid/
-  collapsed-adjacent from URDF topology), out of 1653 pairs in the
+  tool=none  shoulder_ext_length=0.2400 elbow_ext_length=0.2800 shoulder_mount=small elbow_mount=small
+  831 chassis-involving pairs disabled (54 adjacent/always,
+  773 never-colliding over 1000000 random samples, 4 rigid/
+  collapsed-adjacent from URDF topology), out of 1711 pairs in the
   composed robot. "Never" is statistical — see the generator's docstring for
   the trials-vs-pairs convergence on this robot. The rigid/collapsed pairs are
@@ -117,8 +117,6 @@
   <disable_collisions link1="arm_camera_adapter_1" link2="bumper_back_left_1" reason="Never"/>
   <disable_collisions link1="arm_camera_adapter_1" link2="bumper_back_right_1" reason="Never"/>
-  <disable_collisions link1="arm_camera_adapter_1" link2="jetson_mount_1" reason="Never"/>
   <disable_collisions link1="arm_camera_adapter_1" link2="mount_back_left_1" reason="Never"/>
   <disable_collisions link1="arm_camera_adapter_1" link2="mount_back_right_1" reason="Never"/>
-  <disable_collisions link1="arm_camera_adapter_1" link2="orin_simplified_1" reason="Never"/>
   <disable_collisions link1="arm_camera_adapter_1" link2="standoff_back_left_1" reason="Never"/>
   <disable_collisions link1="arm_camera_adapter_1" link2="standoff_back_right_1" reason="Never"/>
@@ -128,8 +126,6 @@
   <disable_collisions link1="arm_camera_wing_1" link2="bumper_back_left_1" reason="Never"/>
   <disable_collisions link1="arm_camera_wing_1" link2="bumper_back_right_1" reason="Never"/>
-  <disable_collisions link1="arm_camera_wing_1" link2="jetson_mount_1" reason="Never"/>
   <disable_collisions link1="arm_camera_wing_1" link2="mount_back_left_1" reason="Never"/>
   <disable_collisions link1="arm_camera_wing_1" link2="mount_back_right_1" reason="Never"/>
-  <disable_collisions link1="arm_camera_wing_1" link2="orin_simplified_1" reason="Never"/>
   <disable_collisions link1="arm_camera_wing_1" link2="standoff_back_left_1" reason="Never"/>
   <disable_collisions link1="arm_camera_wing_1" link2="standoff_back_right_1" reason="Never"/>
@@ -202,5 +198,4 @@
   <disable_collisions link1="arm_end_cap" link2="mount_back_left_1" reason="Never"/>
   <disable_collisions link1="arm_end_cap" link2="mount_back_right_1" reason="Never"/>
-  <disable_collisions link1="arm_end_cap" link2="orin_simplified_1" reason="Never"/>
   <disable_collisions link1="arm_end_cap" link2="standoff_back_left_1" reason="Never"/>
   <disable_collisions link1="arm_end_cap" link2="standoff_back_right_1" reason="Never"/>
@@ -211,9 +206,7 @@
   <disable_collisions link1="arm_forearm_extrusion_1" link2="bumper_back_right_1" reason="Never"/>
   <disable_collisions link1="arm_forearm_extrusion_1" link2="jetson_mount_1" reason="Never"/>
-  <disable_collisions link1="arm_forearm_extrusion_1" link2="link_101_1" reason="Never"/>
   <disable_collisions link1="arm_forearm_extrusion_1" link2="mount_back_left_1" reason="Never"/>
   <disable_collisions link1="arm_forearm_extrusion_1" link2="mount_back_right_1" reason="Never"/>
   <disable_collisions link1="arm_forearm_extrusion_1" link2="orin_simplified_1" reason="Never"/>
-  <disable_collisions link1="arm_forearm_extrusion_1" link2="orp_link101_mount_1" reason="Never"/>
   <disable_collisions link1="arm_forearm_extrusion_1" link2="standoff_back_left_1" reason="Never"/>
   <disable_collisions link1="arm_forearm_extrusion_1" link2="standoff_back_right_1" reason="Never"/>
@@ -395,8 +388,6 @@
   <disable_collisions link1="arm_wrist_camera_v1_1" link2="bumper_back_left_1" reason="Never"/>
   <disable_collisions link1="arm_wrist_camera_v1_1" link2="bumper_back_right_1" reason="Never"/>
-  <disable_collisions link1="arm_wrist_camera_v1_1" link2="jetson_mount_1" reason="Never"/>
   <disable_collisions link1="arm_wrist_camera_v1_1" link2="mount_back_left_1" reason="Never"/>
   <disable_collisions link1="arm_wrist_camera_v1_1" link2="mount_back_right_1" reason="Never"/>
-  <disable_collisions link1="arm_wrist_camera_v1_1" link2="orin_simplified_1" reason="Never"/>
   <disable_collisions link1="arm_wrist_camera_v1_1" link2="standoff_back_left_1" reason="Never"/>
   <disable_collisions link1="arm_wrist_camera_v1_1" link2="standoff_back_right_1" reason="Never"/>
@@ -418,9 +409,7 @@
   <disable_collisions link1="arm_wrist_servo_adapter_1" link2="bumper_back_right_1" reason="Never"/>
   <disable_collisions link1="arm_wrist_servo_adapter_1" link2="jetson_mount_1" reason="Never"/>
-  <disable_collisions link1="arm_wrist_servo_adapter_1" link2="link_101_1" reason="Never"/>
   <disable_collisions link1="arm_wrist_servo_adapter_1" link2="mount_back_left_1" reason="Never"/>
   <disable_collisions link1="arm_wrist_servo_adapter_1" link2="mount_back_right_1" reason="Never"/>
   <disable_collisions link1="arm_wrist_servo_adapter_1" link2="orin_simplified_1" reason="Never"/>
-  <disable_collisions link1="arm_wrist_servo_adapter_1" link2="orp_link101_mount_1" reason="Never"/>
   <disable_collisions link1="arm_wrist_servo_adapter_1" link2="standoff_back_left_1" reason="Never"/>
   <disable_collisions link1="arm_wrist_servo_adapter_1" link2="standoff_back_right_1" reason="Never"/>
