Commit message: changed bumpers, integrated moveit, nicer readme

File: src/base101_arm/base101_arm_moveit_config/config/collisions/parallel.srdf.xacro (robot description, xacro)
@@ -3,8 +3,8 @@
   GENERATED by base101_arm_moveit_config/scripts/gen_collision_matrix.py
   — do not edit by hand.
-  tool=parallel  shoulder_ext_length=0.1400 elbow_ext_length=0.1400 shoulder_mount=small elbow_mount=small
-  855 chassis-involving pairs disabled (54 adjacent/always,
-  797 never-colliding over 1000000 random samples, 4 rigid/
-  collapsed-adjacent from URDF topology), out of 1830 pairs in the
+  tool=parallel  shoulder_ext_length=0.2400 elbow_ext_length=0.2800 shoulder_mount=small elbow_mount=small
+  830 chassis-involving pairs disabled (54 adjacent/always,
+  772 never-colliding over 1000000 random samples, 4 rigid/
+  collapsed-adjacent from URDF topology), out of 1891 pairs in the
   composed robot. "Never" is statistical — see the generator's docstring for
   the trials-vs-pairs convergence on this robot. The rigid/collapsed pairs are
@@ -27,5 +27,4 @@
   <disable_collisions link1="arm_Parallel_gripper_assembly_v1_1" link2="bumper_back_left_1" reason="Never"/>
   <disable_collisions link1="arm_Parallel_gripper_assembly_v1_1" link2="bumper_back_right_1" reason="Never"/>
-  <disable_collisions link1="arm_Parallel_gripper_assembly_v1_1" link2="jetson_mount_1" reason="Never"/>
   <disable_collisions link1="arm_Parallel_gripper_assembly_v1_1" link2="mount_back_left_1" reason="Never"/>
   <disable_collisions link1="arm_Parallel_gripper_assembly_v1_1" link2="mount_back_right_1" reason="Never"/>
@@ -127,8 +126,6 @@
   <disable_collisions link1="arm_camera_adapter_1" link2="bumper_back_left_1" reason="Never"/>
   <disable_collisions link1="arm_camera_adapter_1" link2="bumper_back_right_1" reason="Never"/>
-  <disable_collisions link1="arm_camera_adapter_1" link2="jetson_mount_1" reason="Never"/>
   <disable_collisions link1="arm_camera_adapter_1" link2="mount_back_left_1" reason="Never"/>
   <disable_collisions link1="arm_camera_adapter_1" link2="mount_back_right_1" reason="Never"/>
-  <disable_collisions link1="arm_camera_adapter_1" link2="orin_simplified_1" reason="Never"/>
   <disable_collisions link1="arm_camera_adapter_1" link2="standoff_back_left_1" reason="Never"/>
   <disable_collisions link1="arm_camera_adapter_1" link2="standoff_back_right_1" reason="Never"/>
@@ -138,8 +135,6 @@
   <disable_collisions link1="arm_camera_wing_1" link2="bumper_back_left_1" reason="Never"/>
   <disable_collisions link1="arm_camera_wing_1" link2="bumper_back_right_1" reason="Never"/>
-  <disable_collisions link1="arm_camera_wing_1" link2="jetson_mount_1" reason="Never"/>
   <disable_collisions link1="arm_camera_wing_1" link2="mount_back_left_1" reason="Never"/>
   <disable_collisions link1="arm_camera_wing_1" link2="mount_back_right_1" reason="Never"/>
-  <disable_collisions link1="arm_camera_wing_1" link2="orin_simplified_1" reason="Never"/>
   <disable_collisions link1="arm_camera_wing_1" link2="standoff_back_left_1" reason="Never"/>
   <disable_collisions link1="arm_camera_wing_1" link2="standoff_back_right_1" reason="Never"/>
@@ -210,27 +205,11 @@
   <disable_collisions link1="arm_forearm_extrusion_1" link2="bumper_back_right_1" reason="Never"/>
   <disable_collisions link1="arm_forearm_extrusion_1" link2="jetson_mount_1" reason="Never"/>
-  <disable_collisions link1="arm_forearm_extrusion_1" link2="link_101_1" reason="Never"/>
   <disable_collisions link1="arm_forearm_extrusion_1" link2="mount_back_left_1" reason="Never"/>
   <disable_collisions link1="arm_forearm_extrusion_1" link2="mount_back_right_1" reason="Never"/>
   <disable_collisions link1="arm_forearm_extrusion_1" link2="orin_simplified_1" reason="Never"/>
-  <disable_collisions link1="arm_forearm_extrusion_1" link2="orp_link101_mount_1" reason="Never"/>
   <disable_collisions link1="arm_forearm_extrusion_1" link2="standoff_back_left_1" reason="Never"/>
   <disable_collisions link1="arm_forearm_extrusion_1" link2="standoff_back_right_1" reason="Never"/>
   <disable_collisions link1="arm_forearm_extrusion_1" link2="wheel_back_left_1" reason="Never"/>
   <disable_collisions link1="arm_forearm_extrusion_1" link2="wheel_back_right_1" reason="Never"/>
-  <disable_collisions link1="arm_left_jaw" link2="box_back_1" reason="Never"/>
-  <disable_collisions link1="arm_left_jaw" link2="bumper_back_left_1" reason="Never"/>
-  <disable_collisions link1="arm_left_jaw" link2="bumper_back_right_1" reason="Never"/>
-  <disable_collisions link1="arm_left_jaw" link2="mount_back_left_1" reason="Never"/>
-  <disable_collisions link1="arm_left_jaw" link2="mount_back_right_1" reason="Never"/>
-  <disable_collisions link1="arm_left_jaw" link2="wheel_back_left_1" reason="Never"/>
-  <disable_collisions link1="arm_left_jaw" link2="wheel_back_right_1" reason="Never"/>
-  <disable_collisions link1="arm_right_jaw" link2="box_back_1" reason="Never"/>
-  <disable_collisions link1="arm_right_jaw" link2="bumper_back_left_1" reason="Never"/>
-  <disable_collisions link1="arm_right_jaw" link2="bumper_back_right_1" reason="Never"/>
-  <disable_collisions link1="arm_right_jaw" link2="mount_back_left_1" reason="Never"/>
-  <disable_collisions link1="arm_right_jaw" link2="mount_back_right_1" reason="Never"/>
-  <disable_collisions link1="arm_right_jaw" link2="wheel_back_left_1" reason="Never"/>
-  <disable_collisions link1="arm_right_jaw" link2="wheel_back_right_1" reason="Never"/>
   <disable_collisions link1="arm_servo_base_1" link2="base_link" reason="Never"/>
   <disable_collisions link1="arm_servo_base_1" link2="box_back_1" reason="Never"/>
@@ -408,8 +387,6 @@
   <disable_collisions link1="arm_wrist_camera_v1_1" link2="bumper_back_left_1" reason="Never"/>
   <disable_collisions link1="arm_wrist_camera_v1_1" link2="bumper_back_right_1" reason="Never"/>
-  <disable_collisions link1="arm_wrist_camera_v1_1" link2="jetson_mount_1" reason="Never"/>
   <disable_collisions link1="arm_wrist_camera_v1_1" link2="mount_back_left_1" reason="Never"/>
   <disable_collisions link1="arm_wrist_camera_v1_1" link2="mount_back_right_1" reason="Never"/>
-  <disable_collisions link1="arm_wrist_camera_v1_1" link2="orin_simplified_1" reason="Never"/>
   <disable_collisions link1="arm_wrist_camera_v1_1" link2="standoff_back_left_1" reason="Never"/>
   <disable_collisions link1="arm_wrist_camera_v1_1" link2="standoff_back_right_1" reason="Never"/>
@@ -431,9 +408,7 @@
   <disable_collisions link1="arm_wrist_servo_adapter_1" link2="bumper_back_right_1" reason="Never"/>
   <disable_collisions link1="arm_wrist_servo_adapter_1" link2="jetson_mount_1" reason="Never"/>
-  <disable_collisions link1="arm_wrist_servo_adapter_1" link2="link_101_1" reason="Never"/>
   <disable_collisions link1="arm_wrist_servo_adapter_1" link2="mount_back_left_1" reason="Never"/>
   <disable_collisions link1="arm_wrist_servo_adapter_1" link2="mount_back_right_1" reason="Never"/>
   <disable_collisions link1="arm_wrist_servo_adapter_1" link2="orin_simplified_1" reason="Never"/>
-  <disable_collisions link1="arm_wrist_servo_adapter_1" link2="orp_link101_mount_1" reason="Never"/>
   <disable_collisions link1="arm_wrist_servo_adapter_1" link2="standoff_back_left_1" reason="Never"/>
   <disable_collisions link1="arm_wrist_servo_adapter_1" link2="standoff_back_right_1" reason="Never"/>

File: src/base101_arm/base101_arm_moveit_config/config/collisions/pincopen.srdf.xacro (robot description, xacro)
@@ -3,8 +3,8 @@
   GENERATED by base101_arm_moveit_config/scripts/gen_collision_matrix.py
   — do not edit by hand.
-  tool=pincopen  shoulder_ext_length=0.1400 elbow_ext_length=0.1400 shoulder_mount=small elbow_mount=small
-  872 chassis-involving pairs disabled (54 adjacent/always,
-  814 never-colliding over 1000000 random samples, 4 rigid/
-  collapsed-adjacent from URDF topology), out of 2016 pairs in the
+  tool=pincopen  shoulder_ext_length=0.2400 elbow_ext_length=0.2800 shoulder_mount=small elbow_mount=small
+  835 chassis-involving pairs disabled (54 adjacent/always,
+  777 never-colliding over 1000000 random samples, 4 rigid/
+  collapsed-adjacent from URDF topology), out of 2080 pairs in the
   composed robot. "Never" is statistical — see the generator's docstring for
   the trials-vs-pairs convergence on this robot. The rigid/collapsed pairs are
@@ -117,8 +117,6 @@
   <disable_collisions link1="arm_camera_adapter_1" link2="bumper_back_left_1" reason="Never"/>
   <disable_collisions link1="arm_camera_adapter_1" link2="bumper_back_right_1" reason="Never"/>
-  <disable_collisions link1="arm_camera_adapter_1" link2="jetson_mount_1" reason="Never"/>
   <disable_collisions link1="arm_camera_adapter_1" link2="mount_back_left_1" reason="Never"/>
   <disable_collisions link1="arm_camera_adapter_1" link2="mount_back_right_1" reason="Never"/>
-  <disable_collisions link1="arm_camera_adapter_1" link2="orin_simplified_1" reason="Never"/>
   <disable_collisions link1="arm_camera_adapter_1" link2="standoff_back_left_1" reason="Never"/>
   <disable_collisions link1="arm_camera_adapter_1" link2="standoff_back_right_1" reason="Never"/>
@@ -128,8 +126,6 @@
   <disable_collisions link1="arm_camera_wing_1" link2="bumper_back_left_1" reason="Never"/>
   <disable_collisions link1="arm_camera_wing_1" link2="bumper_back_right_1" reason="Never"/>
-  <disable_collisions link1="arm_camera_wing_1" link2="jetson_mount_1" reason="Never"/>
   <disable_collisions link1="arm_camera_wing_1" link2="mount_back_left_1" reason="Never"/>
   <disable_collisions link1="arm_camera_wing_1" link2="mount_back_right_1" reason="Never"/>
-  <disable_collisions link1="arm_camera_wing_1" link2="orin_simplified_1" reason="Never"/>
   <disable_collisions link1="arm_camera_wing_1" link2="standoff_back_left_1" reason="Never"/>
   <disable_collisions link1="arm_camera_wing_1" link2="standoff_back_right_1" reason="Never"/>
@@ -200,9 +196,7 @@
   <disable_collisions link1="arm_forearm_extrusion_1" link2="bumper_back_right_1" reason="Never"/>
   <disable_collisions link1="arm_forearm_extrusion_1" link2="jetson_mount_1" reason="Never"/>
-  <disable_collisions link1="arm_forearm_extrusion_1" link2="link_101_1" reason="Never"/>
   <disable_collisions link1="arm_forearm_extrusion_1" link2="mount_back_left_1" reason="Never"/>
   <disable_collisions link1="arm_forearm_extrusion_1" link2="mount_back_right_1" reason="Never"/>
   <disable_collisions link1="arm_forearm_extrusion_1" link2="orin_simplified_1" reason="Never"/>
-  <disable_collisions link1="arm_forearm_extrusion_1" link2="orp_link101_mount_1" reason="Never"/>
   <disable_collisions link1="arm_forearm_extrusion_1" link2="standoff_back_left_1" reason="Never"/>
   <disable_collisions link1="arm_forearm_extrusion_1" link2="standoff_back_right_1" reason="Never"/>
@@ -214,40 +208,13 @@
   <disable_collisions link1="arm_pincopen_base_link" link2="mount_back_left_1" reason="Never"/>
   <disable_collisions link1="arm_pincopen_base_link" link2="mount_back_right_1" reason="Never"/>
-  <disable_collisions link1="arm_pincopen_base_link" link2="standoff_back_left_1" reason="Never"/>
-  <disable_collisions link1="arm_pincopen_base_link" link2="standoff_back_right_1" reason="Never"/>
   <disable_collisions link1="arm_pincopen_base_link" link2="wheel_back_left_1" reason="Never"/>
   <disable_collisions link1="arm_pincopen_base_link" link2="wheel_back_right_1" reason="Never"/>
-  <disable_collisions link1="arm_pincopen_left_arm" link2="box_back_1" reason="Never"/>
-  <disable_collisions link1="arm_pincopen_left_arm" link2="bumper_back_left_1" reason="Never"/>
-  <disable_collisions link1="arm_pincopen_left_arm" link2="bumper_back_right_1" reason="Never"/>
   <disable_collisions link1="arm_pincopen_left_arm" link2="mount_back_left_1" reason="Never"/>
   <disable_collisions link1="arm_pincopen_left_arm" link2="mount_back_right_1" reason="Never"/>
-  <disable_collisions link1="arm_pincopen_left_arm" link2="standoff_back_left_1" reason="Never"/>
-  <disable_collisions link1="arm_pincopen_left_arm" link2="standoff_back_right_1" reason="Never"/>
   <disable_collisions link1="arm_pincopen_left_arm" link2="wheel_back_left_1" reason="Never"/>
   <disable_collisions link1="arm_pincopen_left_arm" link2="wheel_back_right_1" reason="Never"/>
-  <disable_collisions link1="arm_pincopen_left_finger" link2="box_back_1" reason="Never"/>
-  <disable_collisions link1="arm_pincopen_left_finger" link2="bumper_back_left_1" reason="Never"/>
-  <disable_collisions link1="arm_pincopen_left_finger" link2="bumper_back_right_1" reason="Never"/>
-  <disable_collisions link1="arm_pincopen_left_finger" link2="mount_back_left_1" reason="Never"/>
-  <disable_collisions link1="arm_pincopen_left_finger" link2="mount_back_right_1" reason="Never"/>
-  <disable_collisions link1="arm_pincopen_left_finger" link2="wheel_back_left_1" reason="Never"/>
-  <disable_collisions link1="arm_pincopen_left_finger" link2="wheel_back_right_1" reason="Never"/>
-  <disable_collisions link1="arm_pincopen_right_arm" link2="box_back_1" reason="Never"/>
-  <disable_collisions link1="arm_pincopen_right_arm" link2="bumper_back_left_1" reason="Never"/>
-  <disable_collisions link1="arm_pincopen_right_arm" link2="bumper_back_right_1" reason="Never"/>
-  <disable_collisions link1="arm_pincopen_right_arm" link2="mount_back_left_1" reason="Never"/>
   <disable_collisions link1="arm_pincopen_right_arm" link2="mount_back_right_1" reason="Never"/>
-  <disable_collisions link1="arm_pincopen_right_arm" link2="standoff_back_left_1" reason="Never"/>
-  <disable_collisions link1="arm_pincopen_right_arm" link2="standoff_back_right_1" reason="Never"/>
   <disable_collisions link1="arm_pincopen_right_arm" link2="wheel_back_left_1" reason="Never"/>
   <disable_collisions link1="arm_pincopen_right_arm" link2="wheel_back_right_1" reason="Never"/>
-  <disable_collisions link1="arm_pincopen_right_finger" link2="box_back_1" reason="Never"/>
-  <disable_collisions link1="arm_pincopen_right_finger" link2="bumper_back_left_1" reason="Never"/>
-  <disable_collisions link1="arm_pincopen_right_finger" link2="bumper_back_right_1" reason="Never"/>
-  <disable_collisions link1="arm_pincopen_right_finger" link2="mount_back_left_1" reason="Never"/>
-  <disable_collisions link1="arm_pincopen_right_finger" link2="mount_back_right_1" reason="Never"/>
-  <disable_collisions link1="arm_pincopen_right_finger" link2="wheel_back_left_1" reason="Never"/>
-  <disable_collisions link1="arm_pincopen_right_finger" link2="wheel_back_right_1" reason="Never"/>
   <disable_collisions link1="arm_servo_base_1" link2="base_link" reason="Never"/>
   <disable_collisions link1="arm_servo_base_1" link2="box_back_1" reason="Never"/>
@@ -425,8 +392,6 @@
   <disable_collisions link1="arm_wrist_camera_v1_1" link2="bumper_back_left_1" reason="Never"/>
   <disable_collisions link1="arm_wrist_camera_v1_1" link2="bumper_back_right_1" reason="Never"/>
-  <disable_collisions link1="arm_wrist_camera_v1_1" link2="jetson_mount_1" reason="Never"/>
   <disable_collisions link1="arm_wrist_camera_v1_1" link2="mount_back_left_1" reason="Never"/>
   <disable_collisions link1="arm_wrist_camera_v1_1" link2="mount_back_right_1" reason="Never"/>
-  <disable_collisions link1="arm_wrist_camera_v1_1" link2="orin_simplified_1" reason="Never"/>
   <disable_collisions link1="arm_wrist_camera_v1_1" link2="standoff_back_left_1" reason="Never"/>
   <disable_collisions link1="arm_wrist_camera_v1_1" link2="standoff_back_right_1" reason="Never"/>
@@ -448,9 +413,7 @@
   <disable_collisions link1="arm_wrist_servo_adapter_1" link2="bumper_back_right_1" reason="Never"/>
   <disable_collisions link1="arm_wrist_servo_adapter_1" link2="jetson_mount_1" reason="Never"/>
-  <disable_collisions link1="arm_wrist_servo_adapter_1" link2="link_101_1" reason="Never"/>
   <disable_collisions link1="arm_wrist_servo_adapter_1" link2="mount_back_left_1" reason="Never"/>
   <disable_collisions link1="arm_wrist_servo_adapter_1" link2="mount_back_right_1" reason="Never"/>
   <disable_collisions link1="arm_wrist_servo_adapter_1" link2="orin_simplified_1" reason="Never"/>
-  <disable_collisions link1="arm_wrist_servo_adapter_1" link2="orp_link101_mount_1" reason="Never"/>
   <disable_collisions link1="arm_wrist_servo_adapter_1" link2="standoff_back_left_1" reason="Never"/>
   <disable_collisions link1="arm_wrist_servo_adapter_1" link2="standoff_back_right_1" reason="Never"/>
